Commit message: some minor updates

File: legged_gym/resources/robots/go2/urdf/go2_nomesh.urdf (robot description, URDF)
Before this commit: robot go2_description, 29 links, 28 joints
Links:
- link FL_calf: geometry collision cylinder length=0.155 radius=0.010
- link FL_foot: geometry collision sphere radius=0.022
- link FL_hip: geometry 
- link FL_thigh: geometry collision box size=0.213 0.0245 0.034
- link FR_calf: geometry collision cylinder length=0.155 radius=0.010
- link FR_foot: geometry collision sphere radius=0.022
- link FR_hip: geometry 
- link FR_thigh: geometry collision box size=0.213 0.0245 0.034
- link RL_calf: geometry collision cylinder length=0.155 radius=0.010
- link RL_foot: geometry collision sphere radius=0.022
- link RL_hip: geometry 
- link RL_thigh: geometry collision box size=0.213 0.0245 0.034
- link RR_calf: geometry collision cylinder length=0.155 radius=0.010
- link RR_foot: geometry collision sphere radius=0.022
- link RR_hip: geometry 
- link RR_thigh: geometry collision box size=0.213 0.0245 0.034
- link base: geometry collision box size=0.3762 0.0935 0.114

File: legged_gym/resources/robots/go2/urdf/go2_nomods_nomesh.urdf (robot description, URDF)
Before this commit: robot go2_description, 29 links, 28 joints
Links:
- link FL_calf: geometry collision cylinder length=0.12 radius=0.012
- link FL_calflower: geometry collision cylinder length=0.065 radius=0.011
- link FL_calflower1: geometry collision cylinder length=0.03 radius=0.0155
- link FL_foot: geometry collision sphere radius=0.022
- link FL_hip: geometry collision cylinder length=0.04 radius=0.046
- link FL_thigh: geometry collision box size=0.213 0.0245 0.034
- link FR_calf: geometry collision cylinder length=0.12 radius=0.013
- link FR_calflower: geometry collision cylinder length=0.065 radius=0.011
- link FR_calflower1: geometry collision cylinder length=0.03 radius=0.0155
- link FR_foot: geometry collision sphere radius=0.022
- link FR_hip: geometry collision cylinder length=0.04 radius=0.046
- link FR_thigh: geometry collision box size=0.213 0.0245 0.034
- link Head_upper: geometry collision cylinder length=0.09 radius=0.05
- link RL_calf: geometry collision cylinder length=0.12 radius=0.013
- link RL_calflower: geometry collision cylinder length=0.065 radius=0.011
- link RL_calflower1: geometry collision cylinder length=0.03 radius=0.0155
- link RL_foot: geometry collision sphere radius=0.022
- link RL_hip: geometry collision cylinder length=0.04 radius=0.046
- link RL_thigh: geometry collision box size=0.213 0.0245 0.034
- link RR_calf: geometry collision cylinder length=0.12 radius=0.013
- link RR_calflower: geometry collision cylinder length=0.065 radius=0.011
- link RR_calflower1: geometry collision cylinder length=0.03 radius=0.0155
- link RR_foot: geometry collision sphere radius=0.022
- link RR_hip: geometry collision cylinder length=0.04 radius=0.046
- link RR_thigh: geometry collision box size=0.213 0.0245 0.034
- link base: geometry collision box size=0.3762 0.0935 0.114
