Commit message: trying simplified mesh

File: legged_gym/resources/robots/go2/urdf/go2.urdf (robot description, URDF)
Before this commit: robot go2_description, 29 links, 28 joints
Links:
- link FL_hip: geometry collision cylinder length=0.04 radius=0.046; visual mesh filename=../meshes/hip_simplified.dae
- link FL_thigh: geometry collision box size=0.213 0.0245 0.034; visual mesh filename=../meshes/thigh_simplified.dae
- link FR_hip: geometry collision cylinder length=0.04 radius=0.046; visual mesh filename=../meshes/hip_simplified.dae
- link FR_thigh: geometry collision box size=0.213 0.0245 0.034; visual mesh filename=../meshes/thigh_mirror_simplified.dae
- link RL_hip: geometry collision cylinder length=0.04 radius=0.046; visual mesh filename=../meshes/hip_simplified.dae
- link RL_thigh: geometry collision box size=0.213 0.0245 0.034; visual mesh filename=../meshes/thigh_simplified.dae
- link RR_hip: geometry collision cylinder length=0.04 radius=0.046; visual mesh filename=../meshes/hip_simplified.dae
- link RR_thigh: geometry collision box size=0.213 0.0245 0.034; visual mesh filename=../meshes/thigh_mirror_simplified.dae
- link base: geometry collision box size=0.3762 0.0935 0.114; visual mesh filename=../meshes/base_simplified.dae

Commit message: radically simplifying collision model

File: legged_gym/resources/robots/go2/urdf/go2.urdf (robot description, URDF)
Before this commit: robot go2_description, 29 links, 28 joints
Links:
- link FL_calf: geometry collision cylinder length=0.155 radius=0.010; visual mesh filename=../meshes/calf.dae
- link FL_calflower: geometry 
- link FL_calflower1: geometry 
- link FL_hip: geometry visual mesh filename=../meshes/hip.dae
- link FR_calf: geometry collision cylinder length=0.155 radius=0.010; visual mesh filename=../meshes/calf_mirror.dae
- link FR_calflower: geometry 
- link FR_calflower1: geometry 
- link FR_foot: geometry collision sphere radius=0.022; visual sphere radius=0.022
- link FR_hip: geometry visual mesh filename=../meshes/hip.dae
- link FR_thigh: geometry collision box size=0.213 0.0245 0.034; visual box size=0.213 0.0245 0.034
- link Head_upper: geometry 
- link RL_calf: geometry collision cylinder length=0.155 radius=0.010; visual mesh filename=../meshes/calf.dae
- link RL_calflower: geometry 
- link RL_calflower1: geometry 
- link RL_hip: geometry visual mesh filename=../meshes/hip.dae
- link RR_calf: geometry collision cylinder length=0.155 radius=0.010; visual mesh filename=../meshes/calf_mirror.dae
- link RR_calflower: geometry 
- link RR_calflower1: geometry 
- link RR_hip: geometry visual mesh filename=../meshes/hip.dae

Commit message: adding new models and infra

File: legged_gym/resources/robots/go2/urdf/go2.urdf (robot description, URDF)
Before this commit: robot go2_description, 29 links, 28 joints
Links:
- link FR_thigh: geometry collision box size=0.213 0.0245 0.034; visual mesh filename=../meshes/thigh_mirror.dae

Commit message: updating collision model

File: legged_gym/resources/robots/go2/urdf/go2.urdf (robot description, URDF)
Before this commit: robot go2_description, 29 links, 28 joints
Links:
- link FL_calf: geometry collision cylinder length=0.24 radius=0.010; visual mesh filename=../meshes/calf.dae
- link FR_calf: geometry collision cylinder length=0.24 radius=0.010; visual mesh filename=../meshes/calf_mirror.dae

Commit message: updating collision model

File: legged_gym/resources/robots/go2/urdf/go2.urdf (robot description, URDF)
Before this commit: robot go2_description, 29 links, 28 joints
Links:
- link RL_calf: geometry collision cylinder length=0.24 radius=0.010; visual mesh filename=../meshes/calf.dae
- link RR_calf: geometry collision cylinder length=0.24 radius=0.010; visual mesh filename=../meshes/calf_mirror.dae

Commit message: removing simplified meshes

File: legged_gym/resources/robots/go2/urdf/go2.urdf (robot description, URDF)
Before this commit: robot go2_description, 29 links, 28 joints
Links:
- link FL_hip: geometry visual mesh filename=../meshes/hip.dae
- link FL_thigh: geometry collision box size=0.213 0.0245 0.034; visual mesh filename=../meshes/thigh.dae
- link FR_hip: geometry visual mesh filename=../meshes/hip.dae
- link FR_thigh: geometry collision box size=0.213 0.0245 0.034; visual mesh filename=../meshes/thigh_mirror.dae
- link RL_hip: geometry visual mesh filename=../meshes/hip.dae
- link RL_thigh: geometry collision box size=0.213 0.0245 0.034; visual mesh filename=../meshes/thigh.dae
- link RR_hip: geometry visual mesh filename=../meshes/hip.dae
- link RR_thigh: geometry collision box size=0.213 0.0245 0.034; visual mesh filename=../meshes/thigh_mirror.dae
- link base: geometry collision box size=0.3762 0.0935 0.114; visual mesh filename=../meshes/base.dae
